File: BumbasiRylan_ElectronicSpeedController/BumbasiRylan_ElectronicSpeedController.kicad_pcb (KiCad board)
At the start: 2 copper layers, 9 parts

Commit message: First revision
Parts:
- added G***: LOGO, Jpeg:logo6'', F.Cu at (125.3, 83.4)
- added G***: LOGO, Jpeg:logo5, F.Cu at (117.6, 82.5)
- added G***: LOGO, Jpeg:logo2, F.Cu at (157.4, 89.1)
- added G***: LOGO, Jpeg:Rylan_logo2, F.Cu at (120.7, 118.4)
- added H1: MountingHole_Pad, MountingHole:MountingHole_3mm_Pad_Via, F.Cu at (157.5, 121.9)
- added H2: MountingHole_Pad, MountingHole:MountingHole_3mm_Pad_Via, F.Cu at (109.2, 121.9)
- added H3: MountingHole_Pad, MountingHole:MountingHole_3mm_Pad_Via, F.Cu at (109.2, 81.3)
- added H4: MountingHole_Pad, MountingHole:MountingHole_3mm_Pad_Via, F.Cu at (157.5, 81.3)
- moved ESC1 9.16 mm to (128.2, 113.4), turned to 0 degrees
- moved LED3 1.76 mm to (109.1, 114.4)
Connections:
- ArduinoNano1 pad 1: Net-(ArduinoNano1-Pad1) -> (no net)
- ArduinoNano1 pad 10: Net-(ArduinoNano1-Pad10) -> (no net)
- ArduinoNano1 pad 11: Net-(ArduinoNano1-Pad11) -> (no net)
- ArduinoNano1 pad 12: Net-(ArduinoNano1-Pad12) -> (no net)
- ArduinoNano1 pad 14: Net-(ArduinoNano1-Pad14) -> (no net)
- ArduinoNano1 pad 15: Net-(ArduinoNano1-Pad15) -> (no net)
- ArduinoNano1 pad 16: Net-(ArduinoNano1-Pad16) -> (no net)
- ArduinoNano1 pad 17: Net-(ArduinoNano1-Pad17) -> (no net)
- ArduinoNano1 pad 18: Net-(ArduinoNano1-Pad18) -> (no net)
- ArduinoNano1 pad 2: Net-(ArduinoNano1-Pad2) -> (no net)
- ArduinoNano1 pad 20: Net-(ArduinoNano1-Pad20) -> (no net)
- ArduinoNano1 pad 21: Net-(ArduinoNano1-Pad21) -> (no net)
- ArduinoNano1 pad 22: Net-(ArduinoNano1-Pad22) -> (no net)
- ArduinoNano1 pad 23: Net-(ArduinoNano1-Pad23) -> (no net)
- ArduinoNano1 pad 24: Net-(ArduinoNano1-Pad24) -> (no net)
- ArduinoNano1 pad 25: Net-(ArduinoNano1-Pad25) -> (no net)
- ArduinoNano1 pad 26: Net-(ArduinoNano1-Pad26) -> (no net)
- ArduinoNano1 pad 28: Net-(ArduinoNano1-Pad28) -> (no net)
- ArduinoNano1 pad 3: Net-(ArduinoNano1-Pad3) -> (no net)
- ArduinoNano1 pad 30: Net-(ArduinoNano1-Pad30) -> (no net)
- ArduinoNano1 pad 8: Net-(ArduinoNano1-Pad8) -> (no net)
- ArduinoNano1 pad 9: Net-(ArduinoNano1-Pad9) -> (no net)
- ESC1 pad 2: Net-(ESC1-Pad2) -> (no net)
Routing:
- net /D10(PWM): track 16.5 -> 6.71 mm
- net Net-(LED3-Pad2): track 11.7 -> 9.86 mm
Other:
- board outline added: 58.4 x 50.8 mm
- board text added: "ESC Tester SDSU Mechatronics Designed by: Rylan Bumbasi"
- board text added: "GREEN"
- board text added: "RED"
- board text added: "YELLOW"
