File: PCB/kicad intro project.kicad_pcb (KiCad board)
At the start: 2 copper layers, 5 parts, among them SW1 SW_SPST

Commit message: project complete
Other:
- board outline added: 41.9 x 50.8 mm
Changed lines of the file:
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@@
   (general
     (thickness 1.6)
-    (drawings 0)
+    (drawings 4)
     (tracks 17)
     (zones 0)
@@
       (usegerberattributes false)
       (usegerberadvancedattributes false)
-      (creategerberjobfile false)
+      (creategerberjobfile true)
       (excludeedgelayer true)
       (linewidth 0.100000)
@@
       (outputformat 1)
       (mirror false)
-      (drillshape 1)
+      (drillshape 0)
       (scaleselection 1)
       (outputdirectory ""))
@@
     )
   )
+  (gr_line (start 135.89 59.69) (end 135.89 110.49) (layer Edge.Cuts) (width 0.05))
+  (gr_line (start 93.98 59.69) (end 135.89 59.69) (layer Edge.Cuts) (width 0.05))
+  (gr_line (start 93.98 110.49) (end 135.89 110.49) (layer Edge.Cuts) (width 0.05))
+  (gr_line (start 93.98 59.69) (end 93.98 110.49) (layer Edge.Cuts) (width 0.05))
   (segment (start 124.58 74.93) (end 125.73 74.93) (width 0.25) (layer F.Cu) (net 7))
   (segment (start 123.19 76.32) (end 124.58 74.93) (width 0.25) (layer F.Cu) (net 7))
